File: PSU - Transformer.kicad_pcb (KiCad board)
At the start: 2 copper layers, 160 x 111.8 mm, 16 parts, among them J1 220V, J2 Header_1x03, J3 Header_1x03, J4 Header_1x03, J5 Header_1x03, T1 +/-12V

Commit message: Fixed library dependencies
Parts:
- D1, D2: footprint MojaBiblioteka:Diode_Bridge_18.5x5.5 -> KraakenStuff:Diode_Bridge_18.5x5.5
- F1, F2: footprint Fuse_Holders_and_Fuses:Fuseholder5x20_horiz_SemiClosed_Casing10x25mm -> KraakenStuff:Fuseholder5x20_horiz_SemiClosed_Casing10x25mm
- J1: footprint MojaBiblioteka:BLOK TERMINAL 2 KONTAKTA -> KraakenStuff:Terminal 2 contacts
- J2, J3, J4, J5: value Header_1x03 -> Conn_01x03_Male; footprint MojaBiblioteka:Klema x3 -> KraakenStuff:Klema x3
- T1: footprint MojaBiblioteka:TRAFO TORUSNI 220V 150VA 2x12V -> KraakenStuff:Toroidal transformer 220V 150VA 2x12V
- moved J1 0.13 mm to (86.3, 48.2), turned to 90 degrees
- moved J3 0.05 mm to (223.5, 71.1), turned to 270 degrees
- turned J5 to 270 degrees
- turned J2 to 270 degrees
- turned J4 to 270 degrees
Connections:
- J1 pad 1: Net-(F2-Pad2) -> Net-(F1-Pad2)
- J1 pad 2: Net-(F1-Pad2) -> Net-(F2-Pad2)
- J2 pad 1: -12_IN -> +12_IN
- J2 pad 3: +12_IN -> -12_IN
- J3 pad 1: -12_IN -> +12_IN
- J3 pad 3: +12_IN -> -12_IN
- J4 pad 1: -12_IN -> +12_IN
- J4 pad 3: +12_IN -> -12_IN
- J5 pad 1: -12_IN -> +12_IN
- J5 pad 3: +12_IN -> -12_IN

Commit message: Finished. First round of testing passed
Other:
- board text added: "KraakenStuff PSU (main board) v.0.2"
Changed lines of the file:
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@@
   (general
     (thickness 1.6)
-    (drawings 13)
+    (drawings 14)
     (tracks 74)
     (zones 0)
@@
       (drillshape 0)
       (scaleselection 1)
-      (outputdirectory "Gerber Trans/"))
+      (outputdirectory "Gerber/"))
   )
   (net 0 "")
@@
   (module "KraakenStuff:Klema x3" (layer F.Cu)
     (at 223.52 48.2346 270)
-    (fp_text reference J2 (at 0 7.62 270) (layer F.SilkS)
+    (fp_text reference J2 (at 0 6.1976 270) (layer F.SilkS)
       (effects (font (size 1 1) (thickness 0.15)))
     )
@@
   (module "KraakenStuff:Klema x3" (layer F.Cu)
     (at 223.52 71.0692 270)
-    (fp_text reference J3 (at 0 7.62 270) (layer F.SilkS)
+    (fp_text reference J3 (at 0 6.1976 270) (layer F.SilkS)
       (effects (font (size 1 1) (thickness 0.15)))
     )
@@
   (module "KraakenStuff:Klema x3" (layer F.Cu)
     (at 223.52 93.98 270)
-    (fp_text reference J4 (at 0 7.62 270) (layer F.SilkS)
+    (fp_text reference J4 (at 0 6.1976 270) (layer F.SilkS)
       (effects (font (size 1 1) (thickness 0.15)))
     )
@@
   )
   (module "KraakenStuff:Klema x3" (layer F.Cu)
-    (at 223.4946 116.8146 270)
-    (fp_text reference J5 (at 0 7.62 270) (layer F.SilkS)
+    (at 223.4946 116.814599 270)
+    (fp_text reference J5 (at -0.0254 6.1722 270) (layer F.SilkS)
       (effects (font (size 1 1) (thickness 0.15)))
     )
@@
     (pad "" np_thru_hole circle (at 0 0) (size 8 8) (drill 5.2) (layers *.Cu *.Mask))
   )
+  (gr_text "KraakenStuff\nPSU (main board) v.0.2" (at 216.5858 82.524601 90) (layer B.SilkS)
+    (effects (font (size 1.5 1.5) (thickness 0.3)) (justify mirror))
+  )
   (gr_arc (start 223.52 33.02) (end 228.6 33.02) (angle -90) (layer Edge.Cuts) (width 0.1))
   (gr_arc (start 223.52 134.62) (end 223.52 139.7) (angle -90) (layer Edge.Cuts) (width 0.1))
@@
   (gr_line (start 223.52 139.7) (end 73.66 139.7) (layer Edge.Cuts) (width 0.1))
   (gr_line (start 73.66 27.94) (end 223.52 27.94) (layer Edge.Cuts) (width 0.1))
-  (gr_text "-12V GND +12V" (at 214.63 116.84 90) (layer F.SilkS)
+  (gr_text "-12V GND +12V" (at 215.519 116.8146 90) (layer F.SilkS)
     (effects (font (size 1 1) (thickness 0.25)))
   )
-  (gr_text "-12V GND +12V" (at 213.36 93.98 90) (layer F.SilkS)
+  (gr_text "-12V GND +12V" (at 215.519 93.98 90) (layer F.SilkS)
     (effects (font (size 1 1) (thickness 0.25)))
   )
-  (gr_text "-12V GND +12V" (at 213.36 71.12 90) (layer F.SilkS)
+  (gr_text "-12V GND +12V" (at 215.519 71.12 90) (layer F.SilkS)
     (effects (font (size 1 1) (thickness 0.25)))
   )
-  (gr_text "-12V GND +12V" (at 213.36 48.26 90) (layer F.SilkS)
+  (gr_text "-12V GND +12V" (at 215.519 48.26 90) (layer F.SilkS)
     (effects (font (size 1 1) (thickness 0.25)))
   )

Commit message: Adapted for KiCad6. Also fixed an error in silkscreen for the filter
Other:
- net class 220V removed
- net class Default removed
